File: patch/patch.kicad_sch (KiCad schematic)
At the start: 22 parts, among them J1 Eurorack_Mono_Jack, J2 Eurorack_Mono_Jack, J3 Eurorack_Mono_Jack_No_S, J4 Eurorack_Mono_Jack_No_S, J5 Eurorack_Power, U1 OPA4991

Commit message: Patch: Start of feedback, more channels
Addressed some feedback, switched to TSSOP/0603 to get better margins.
Started on more channels to make sure the jack and part placement is OK.
Parts:
- added J1: In 3: A, winterbloom:AudioJack_WQP518MA_Compact_S, symbol winterbloom:Eurorack_Mono_Jack
- added J1: In 2: A, winterbloom:AudioJack_WQP518MA_Compact_S, symbol winterbloom:Eurorack_Mono_Jack
- added J1: In 4: A, winterbloom:AudioJack_WQP518MA_Compact_S, symbol winterbloom:Eurorack_Mono_Jack
- added J2: In 3: B, winterbloom:AudioJack_WQP518MA_Compact_S, symbol winterbloom:Eurorack_Mono_Jack
- added J2: In 4: B, winterbloom:AudioJack_WQP518MA_Compact_S, symbol winterbloom:Eurorack_Mono_Jack
- added J2: In 2: B, winterbloom:AudioJack_WQP518MA_Compact_S, symbol winterbloom:Eurorack_Mono_Jack
- added J3: Out 4: max(A,0)+min(B,0), winterbloom:AudioJack_WQP518MA_No_S, symbol winterbloom:Eurorack_Mono_Jack_No_S
- added J3: Out 3: max(A,B), winterbloom:AudioJack_WQP518MA_No_S, symbol winterbloom:Eurorack_Mono_Jack_No_S
- added J3: Out 2: (A+B)/2, winterbloom:AudioJack_WQP518MA_No_S, symbol winterbloom:Eurorack_Mono_Jack_No_S
- added J4: Out 4: min(A,0)+max(B,0), winterbloom:AudioJack_WQP518MA_No_S, symbol winterbloom:Eurorack_Mono_Jack_No_S
- added J4: Out 3: min(A,B), winterbloom:AudioJack_WQP518MA_No_S, symbol winterbloom:Eurorack_Mono_Jack_No_S
- added J4: Out 2: (2A+B)/3, winterbloom:AudioJack_WQP518MA_No_S, symbol winterbloom:Eurorack_Mono_Jack_No_S
- added R1 (x3), R2 (x4), R3 (x3), R4 (x3), R5 (x2), R6 (x2), R7 (x2), R8 (x2): 10k, winterbloom:R_0603_HandSolder, symbol Device:R
- added R10 (x3), R9 (x3): 51R, winterbloom:R_0603_HandSolder, symbol Device:R
- added U1 (x3): OPA4991, Package_SO:TSSOP-14_4.4x5mm_P0.65mm, symbol winterbloom:OPA4991
- C1, C2: value 100nF -> 100n; footprint Capacitor_SMD:C_0805_2012Metric_Pad1.18x1.45mm_HandSolder -> winterbloom:C_0603_HandSolder; Rating (none) -> 25V/10%/X7R
- C10, C9: value 10uF -> 10u; footprint Capacitor_SMD:C_0805_2012Metric_Pad1.18x1.45mm_HandSolder -> winterbloom:C_0805_HandSolder; Rating (none) -> 25V/10%/X7R
- D1, D2: value D_Schottky -> 30V; MPN (none) -> MBR0530T1G; Rating (none) -> 500mA
- J1: value Eurorack_Mono_Jack -> In 1: A
- J2: value Eurorack_Mono_Jack -> In 1: B
- J3: value Eurorack_Mono_Jack_No_S -> Out 1: A+B
- J4: value Eurorack_Mono_Jack_No_S -> Out 1: A-B
- R1, R2, R3, R4, R5, R6, R7, R8: footprint Resistor_SMD:R_0805_2012Metric_Pad1.20x1.40mm_HandSolder -> winterbloom:R_0603_HandSolder; Rating (none) -> 100mW/1%/Thin
- R10, R9: value 51 -> 51R; footprint Resistor_SMD:R_0805_2012Metric_Pad1.20x1.40mm_HandSolder -> winterbloom:R_0603_HandSolder; Rating (none) -> 100mW/1%/Thin
- U1: footprint Package_SO:SOIC-14_3.9x8.7mm_P1.27mm -> Package_SO:TSSOP-14_4.4x5mm_P0.65mm
Connections:
- net GND: now also J1.S (Sleeve), J1.S (Sleeve), J1.S (Sleeve), J2.S (Sleeve), J2.S (Sleeve), J2.S (Sleeve), R7.1, R7.1, R8.1, R8.1
- net at J1.T (Tip), U1.5 (+): now also J1.TN (Tip_normalize)
- new net: R3.2, R4.1, U1.3 (+) (x3)
- new net: R1.2, R4.2, U1.6 (-), U1.7 (x3)
- new net: R1.1, R8.2, U1.12 (+) (x2)
- new net: R2.1, R5.1, U1.13 (-) (x2)
- new net: R5.2, R9.1, U1.14 (x2)
- new net: J4.T (Tip), R9.2 (x3)
- new net: J1.T (Tip), J2.TN (Tip_normalize), U1.5 (+)
- new net: J2.T (Tip), U1.10 (+) (x3)
- new net: R2.2, R3.1, U1.8, U1.9 (-) (x3)
- new net: R2.1, R2.2
- new net: R10.1, U1.1, U1.2 (-)
- new net: J3.T (Tip), R10.2 (x3)
- new net: J1.T (Tip), J1.TN (Tip_normalize), J2.TN (Tip_normalize), U1.5 (+) (x2)
- new net: R6.1, R7.2, U1.2 (-) (x2)
- new net: R10.1, R6.2, U1.1 (x2)
- new net: R1.1, R2.1, U1.12 (+)
- new net: R9.1, U1.13 (-), U1.14
- no-connect marks 2 -> 8
Other:
- note removed: "Resistors are 0.1%"
- moved on the sheet: C1, C10, C2, C9, D1, D2, J1, J2, J3, J4, J5, R1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
